Commit message: resolved lidar publishing error

File: vertical_farm_isaac_ros/src/rur5/urdf/ridgeback_ur5.urdf (robot description, URDF)
Before this commit: robot ridgeback_ur5, 11 links, 10 joints
Links:
- removed link TiM_781
- added link tim781; visual cylinder length=0.05 radius=0.05
Joints:
- joint base_lidar: child TiM_781 -> tim781
